File: ProjectEAGLE/fonte_schema.sch (EAGLE design)
At the start: 10 parts, among them T1 2N3904

Commit message: Finalizando
Parts:
- removed C2: 750u, rcl:C-USC0805
- removed D5: 13v, diode:ZENER-DIODEDO35Z10
- removed R3: 2.2k, rcl:R-US_R0805
- removed R5: 120, rcl:R-US_R0805
- removed TR1: 15V, inductor-neosid:SM-T4
- added C1: 750u, rcl:C-US025-025X050
- added D1: 13v, diode:BZD23
- added JP2: 3-12V, pinhead:PINHD-1X2
- added R1: 330, rcl:R-EU_0204/7
- JP1: value 127V -> 15V
- R2: value 330 -> 2.2k; device rcl:R-US_R0805 -> rcl:R-EU_0204/7
- R4: value 4.7k -> 5k
Connections:
- removed net N$10: JP1.2, TR1.E1
- removed net N$9: JP1.1, TR1.A1
- net N$1: now also JP2.2, T1.E; no longer B1.-, C2.2, D5.A, R3.1, R5.1
- net N$2: now also JP1.1; no longer TR1.A2
- net N$3: now also C1.1, R1.1; no longer C2.1, R2.1
- net N$4: now also D1.C, R1.2; no longer D5.C, R2.2
- net N$5: now also JP1.2; no longer TR1.E2
- net N$7: now also R2.2; no longer R3.2
- net N$8: now also B1.-, C1.2, D1.A, JP2.1, R2.1; no longer R5.2, T1.E
Other:
- moved on the sheet: JP1
